File: ai03-pcb-guide.sch (KiCad schematic (older format))
At the start: 24 parts, among them SW1 SW_Push, U1 ATmega32U4-AU, Y1 10MHz

Commit message: PCB layout & traces
Parts:
- MX1, MX4: footprint MX_Alps_Hybrid:MX-1U-NoLED -> MX_Alps_Hybrid:MX-1U
- MX2: renamed from MX3; footprint MX_Alps_Hybrid:MX-1U-NoLED -> MX_Alps_Hybrid:MX-1U
- MX3: renamed from MX2; footprint MX_Alps_Hybrid:MX-1U-NoLED -> MX_Alps_Hybrid:MX-1U
- renumbered D3 to D2, D2 to D3
Connections:
- net COL0: now also U1.28 (PB4)
- net COL1: now also U1.29 (PB5)
- net ROW0: now also U1.27 (PD7)
- net ROW1: now also U1.30 (PB6)
Changed lines of the file:
@@
 F 0 "MX1" H 9033 4673 60  0000 C CNN
 F 1 "MX-NoLED" H 9033 4599 20  0000 C CNN
-F 2 "MX_Alps_Hybrid:MX-1U-NoLED" H 8375 4425 60  0001 C CNN
+F 2 "MX_Alps_Hybrid:MX-1U" H 8375 4425 60  0001 C CNN
 F 3 "" H 8375 4425 60  0001 C CNN
 	1    9000 4450
@@
 	8950 4600 8850 4600
 $Comp
-L MX_Alps_Hybrid:MX-NoLED MX3
+L MX_Alps_Hybrid:MX-NoLED MX2
 U 1 1 5F32E5D2
 P 9700 4450
-F 0 "MX3" H 9733 4673 60  0000 C CNN
+F 0 "MX2" H 9733 4673 60  0000 C CNN
 F 1 "MX-NoLED" H 9733 4599 20  0000 C CNN
-F 2 "MX_Alps_Hybrid:MX-1U-NoLED" H 9075 4425 60  0001 C CNN
+F 2 "MX_Alps_Hybrid:MX-1U" H 9075 4425 60  0001 C CNN
 F 3 "" H 9075 4425 60  0001 C CNN
 	1    9700 4450
@@
 $EndComp
 $Comp
-L Device:D_Small D3
+L Device:D_Small D2
 U 1 1 5F32F703
 P 9550 4700
-F 0 "D3" H 9550 4800 50  0000 R CNN
+F 0 "D2" H 9550 4800 50  0000 R CNN
 F 1 "D_Small" H 9900 4800 50  0000 R CNN
 F 2 "Diode_SMD:D_SOD-123" V 9550 4700 50  0001 C CNN
@@
 	9550 4600 9650 4600
 $Comp
-L MX_Alps_Hybrid:MX-NoLED MX2
+L MX_Alps_Hybrid:MX-NoLED MX3
 U 1 1 5F332C02
 P 9000 5200
-F 0 "MX2" H 9033 5423 60  0000 C CNN
+F 0 "MX3" H 9033 5423 60  0000 C CNN
 F 1 "MX-NoLED" H 9033 5349 20  0000 C CNN
-F 2 "MX_Alps_Hybrid:MX-1U-NoLED" H 8375 5175 60  0001 C CNN
+F 2 "MX_Alps_Hybrid:MX-1U" H 8375 5175 60  0001 C CNN
 F 3 "" H 8375 5175 60  0001 C CNN
 	1    9000 5200
@@
 $EndComp
 $Comp
-L Device:D_Small D2
+L Device:D_Small D3
 U 1 1 5F333941
 P 8850 5450
-F 0 "D2" H 8850 5550 50  0000 R CNN
+F 0 "D3" H 8850 5550 50  0000 R CNN
 F 1 "D_Small" H 9200 5550 50  0000 R CNN
 F 2 "Diode_SMD:D_SOD-123" V 8850 5450 50  0001 C CNN
@@
 F 0 "MX4" H 9733 5423 60  0000 C CNN
 F 1 "MX-NoLED" H 9733 5349 20  0000 C CNN
-F 2 "MX_Alps_Hybrid:MX-1U-NoLED" H 9075 5175 60  0001 C CNN
+F 2 "MX_Alps_Hybrid:MX-1U" H 9075 5175 60  0001 C CNN
 F 3 "" H 9075 5175 60  0001 C CNN
 	1    9700 5200
@@
 Text GLabel 9850 4000 1    50   Input ~ 0
 COL1
+Text GLabel 5000 2950 2    50   Input ~ 0
+COL0
+Text GLabel 5000 3050 2    50   Input ~ 0
+COL1
+Text GLabel 5000 4450 2    50   Input ~ 0
+ROW0
+Text GLabel 5000 3150 2    50   Input ~ 0
+ROW1
 $EndSCHEMATC
