File: ai03-pcb-guide.kicad_pcb (KiCad board)
At the start: 2 copper layers, 84.1 x 38.1 mm, 24 parts, among them SW1 SW_Push, U1 ATmega32U4-AU, Y1 10MHz

Commit message: Generated Gerber files and finalized pcb
Routing:
- added copper zone on B.Cu, net GND
Other:
- board text added: "The Brains"
Changed lines of the file:
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@@
   (general
     (thickness 1.6)
-    (drawings 8)
+    (drawings 9)
     (tracks 230)
     (zones 0)
@@
     (solder_mask_min_width 0.25)
     (aux_axis_origin 0 0)
-    (visible_elements FFFFFF7F)
+    (visible_elements 7FFFFFFF)
     (pcbplotparams
-      (layerselection 0x010fc_ffffffff)
+      (layerselection 0x010f0_ffffffff)
       (usegerberextensions false)
       (usegerberattributes false)
@@
       (plotinvisibletext false)
       (padsonsilk false)
-      (subtractmaskfromsilk false)
+      (subtractmaskfromsilk true)
       (outputformat 1)
       (mirror false)
-      (drillshape 1)
+      (drillshape 0)
       (scaleselection 1)
       (outputdirectory ""))
@@
     )
   )
+  (gr_text "The Brains" (at 66.675 80.16875) (layer B.SilkS)
+    (effects (font (size 1 1) (thickness 0.15)) (justify mirror))
+  )
   (gr_line (start 35.71875 85.725) (end 115.09375 85.725) (layer Edge.Cuts) (width 0.05))
   (gr_line (start 115.09375 47.625) (end 35.71875 47.625) (layer Edge.Cuts) (width 0.05))
@@
   (gr_arc (start 115.09375 83.34375) (end 115.09375 85.725) (angle -90) (layer Edge.Cuts) (width 0.05))
   (gr_arc (start 115.09375 50.00625) (end 117.475 50.00625) (angle -90) (layer Edge.Cuts) (width 0.05))
-  (segment (start 85.09 54.61) (end 85.09 58.674) (width 0.254) (layer B.Cu) (net 13))
-  (segment (start 85.09 70.739) (end 85.09 73.66) (width 0.254) (layer B.Cu) (net 13))
-  (via (at 85.09 58.674) (size 0.8) (drill 0.4) (layers F.Cu B.Cu) (net 13))
-  (via (at 85.09 70.739) (size 0.8) (drill 0.4) (layers F.Cu B.Cu) (net 13))
   (segment (start 53.654 70.80425) (end 54.483 69.97525) (width 0.381) (layer B.Cu) (net 1))
   (segment (start 46.00575 70.80425) (end 53.654 70.80425) (width 0.381) (layer B.Cu) (net 1))
@@
   (segment (start 41.23075 54.723) (end 35.687 60.26675) (width 0.381) (layer B.Cu) (net 12))
   (segment (start 41.23075 53.848) (end 41.23075 54.723) (width 0.381) (layer B.Cu) (net 12))
+  (segment (start 85.09 54.61) (end 85.09 58.674) (width 0.254) (layer B.Cu) (net 13))
+  (segment (start 85.09 70.739) (end 85.09 73.66) (width 0.254) (layer B.Cu) (net 13))
+  (via (at 85.09 58.674) (size 0.8) (drill 0.4) (layers F.Cu B.Cu) (net 13))
+  (via (at 85.09 70.739) (size 0.8) (drill 0.4) (layers F.Cu B.Cu) (net 13))
   (via (at 85.09 66.348) (size 0.8) (drill 0.4) (layers F.Cu B.Cu) (net 13))
   (segment (start 85.09 66.167) (end 85.09 66.348) (width 0.254) (layer F.Cu) (net 13))
@@
   (segment (start 71.99325 76.073) (end 73.533 74.53325) (width 0.254) (layer B.Cu) (net 20))
   (segment (start 71.40575 76.073) (end 71.99325 76.073) (width 0.254) (layer B.Cu) (net 20))
-  (segment (start 46.48075 53.848) (end 46.48075 49.348) (width 0.254) (layer B.Cu) (net 43))
   (segment (start 45.37675 49.348) (end 39.18075 49.348) (width 0.254) (layer B.Cu) (net 43))
   (segment (start 46.48075 49.348) (end 45.37675 49.348) (width 0.254) (layer B.Cu) (net 43))
-  (segment (start 39.18075 50.952) (end 39.18075 53.848) (width 0.254) (layer B.Cu) (net 43))
-  (segment (start 39.18075 49.348) (end 39.18075 50.952) (width 0.254) (layer B.Cu) (net 43))
+  (segment (start 39.18075 49.348) (end 39.18075 53.848) (width 0.254) (layer B.Cu) (net 43))
+  (segment (start 46.48075 50.952) (end 46.48075 53.848) (width 0.254) (layer B.Cu) (net 43))
+  (segment (start 46.48075 49.348) (end 46.48075 50.952) (width 0.254) (layer B.Cu) (net 43))
+  (zone (net 1) (net_name GND) (layer B.Cu) (hatch edge 0.508)
+    (connect_pads (clearance 0.508))
+    (min_thickness 0.254)
+    (fill yes (arc_segments 32) (thermal_gap 0.508) (thermal_bridge_width 0.508))
+    (polygon
+      (pts
+        (xy 33.3375 47.625) (xy 33.3375 85.725) (xy 79.375 85.725) (xy 79.375 47.625)
+      )
+    )
+  )
 )

Commit message: Remade gerbers
Other:
- board text added: "Elsbree Enterprises"
- board text removed: "The Brains"
Changed lines of the file:
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@@
       (effects (font (size 1 1) (thickness 0.15)) (justify mirror))
     )
-    (fp_text value ATmega32U4-AU (at 0 -7.45) (layer B.Fab)
+    (fp_text value ATmega32U4-AU (at 0 -8.001) (layer B.SilkS)
       (effects (font (size 1 1) (thickness 0.15)) (justify mirror))
     )
@@
     (tags resistor)
     (attr smd)
-    (fp_text reference R4 (at 0 1.65) (layer B.SilkS)
+    (fp_text reference R4 (at -2.9995 0.127) (layer B.SilkS)
       (effects (font (size 1 1) (thickness 0.15)) (justify mirror))
     )
@@
     (tags capacitor)
     (attr smd)
-    (fp_text reference C6 (at 0 1.65 90) (layer B.SilkS)
+    (fp_text reference C6 (at -2.93775 -0.28575 90) (layer B.SilkS)
       (effects (font (size 1 1) (thickness 0.15)) (justify mirror))
     )
@@
     (tags capacitor)
     (attr smd)
-    (fp_text reference C3 (at 0 1.65 90) (layer B.SilkS)
+    (fp_text reference C3 (at 2.4915 0.03175 90) (layer B.SilkS)
       (effects (font (size 1 1) (thickness 0.15)) (justify mirror))
     )
@@
     (tags capacitor)
     (attr smd)
-    (fp_text reference C2 (at 0 1.65) (layer B.SilkS)
+    (fp_text reference C2 (at -2.49325 0.127) (layer B.SilkS)
       (effects (font (size 1 1) (thickness 0.15)) (justify mirror))
     )
@@
     (tags capacitor)
     (attr smd)
-    (fp_text reference C1 (at 0 1.65 90) (layer B.SilkS)
+    (fp_text reference C1 (at -2.906 0.28575 90) (layer B.SilkS)
       (effects (font (size 1 1) (thickness 0.15)) (justify mirror))
     )
@@
     )
   )
-  (gr_text "The Brains" (at 66.675 80.16875) (layer B.SilkS)
-    (effects (font (size 1 1) (thickness 0.15)) (justify mirror))
+  (gr_text "Elsbree Enterprises" (at 43.65625 82.55) (layer F.SilkS)
+    (effects (font (size 1 1) (thickness 0.15)))
   )
   (gr_line (start 35.71875 85.725) (end 115.09375 85.725) (layer Edge.Cuts) (width 0.05))
